File: Stepper_Board/StepperBoard.sch (KiCad schematic (older format))
At the start: 6 parts

Commit message: Testsoftware for ImageProcessing in c programmiert
Parts:
- PS101: renamed from PS?; symbol Pick_n_Place:MEANWELL-MPM-90 -> StepperBoard-rescue:MEANWELL-MPM-90-Pick_n_Place
- gave numbers to parts that had none: 5
Changed lines of the file:
@@
 EESchema Schematic File Version 4
-LIBS:Pick_n_Place-cache
+LIBS:StepperBoard-cache
 EELAYER 26 0
 EELAYER END
 $Descr A4 11693 8268
 encoding utf-8
-Sheet 1 3
+Sheet 1 5
 Title ""
 Date ""
@@
 $EndSheet
 $Comp
-L Connector:Screw_Terminal_01x04 J?
+L Connector:Screw_Terminal_01x04 J105
 U 1 1 5FBFBC6F
 P 9450 5500
-F 0 "J?" H 9530 5537 50  0000 L CNN
+F 0 "J105" H 9530 5537 50  0000 L CNN
 F 1 "Screw_Terminal_01x04" H 9530 5446 50  0000 L CNN
 F 2 "TerminalBlock_RND:TerminalBlock_RND_205-00047_1x04_P5.00mm_Horizontal" H 9450 5500 50  0001 C CNN
@@
 	8800 5700 9250 5700
 $Comp
-L Connector:Screw_Terminal_01x04 J?
+L Connector:Screw_Terminal_01x04 J104
 U 1 1 5FBFC3D6
 P 9450 4200
-F 0 "J?" H 9530 4237 50  0000 L CNN
+F 0 "J104" H 9530 4237 50  0000 L CNN
 F 1 "Screw_Terminal_01x04" H 9530 4146 50  0000 L CNN
 F 2 "TerminalBlock_RND:TerminalBlock_RND_205-00047_1x04_P5.00mm_Horizontal" H 9450 4200 50  0001 C CNN
@@
 	8800 4400 9250 4400
 $Comp
-L Connector:Screw_Terminal_01x04 J?
+L Connector:Screw_Terminal_01x04 J103
 U 1 1 5FBFC7E1
 P 9450 2750
-F 0 "J?" H 9530 2787 50  0000 L CNN
+F 0 "J103" H 9530 2787 50  0000 L CNN
 F 1 "Screw_Terminal_01x04" H 9530 2696 50  0000 L CNN
 F 2 "TerminalBlock_RND:TerminalBlock_RND_205-00047_1x04_P5.00mm_Horizontal" H 9450 2750 50  0001 C CNN
@@
 	8800 2950 9250 2950
 $Comp
-L Connector:Screw_Terminal_01x04 J?
+L Connector:Screw_Terminal_01x04 J102
 U 1 1 5FBFCACB
 P 9450 1350
-F 0 "J?" H 9530 1387 50  0000 L CNN
+F 0 "J102" H 9530 1387 50  0000 L CNN
 F 1 "Screw_Terminal_01x04" H 9530 1296 50  0000 L CNN
 F 2 "TerminalBlock_RND:TerminalBlock_RND_205-00047_1x04_P5.00mm_Horizontal" H 9450 1350 50  0001 C CNN
@@
 	8800 1550 9250 1550
 $Comp
-L Connector:Screw_Terminal_01x02 J?
+L Connector:Screw_Terminal_01x02 J101
 U 1 1 5FBE8C83
 P 950 1250
-F 0 "J?" H 870 835 50  0000 C CNN
+F 0 "J101" H 870 835 50  0000 C CNN
 F 1 "Screw_Terminal_01x02" H 870 926 50  0000 C CNN
 F 2 "TerminalBlock_RND:TerminalBlock_RND_205-00045_1x02_P5.00mm_Horizontal" H 950 1250 50  0001 C CNN
@@
 $EndComp
 $Comp
-L Pick_n_Place:MEANWELL-MPM-90 PS?
+L StepperBoard-rescue:MEANWELL-MPM-90-Pick_n_Place PS101
 U 1 1 5FC0E18E
 P 1900 1200
-F 0 "PS?" H 1900 1567 50  0000 C CNN
+F 0 "PS101" H 1900 1567 50  0000 C CNN
 F 1 "MEANWELL-MPM-90" H 1900 1476 50  0000 C CNN
 F 2 "pick_n_place:MEANWELL-MPM-90" H 1900 850 50  0001 C CNN
@@
 	1150 1300 1150 1250
 $Comp
-L power:+24V #PWR?
+L power:+24V #PWR0112
 U 1 1 5FC10E36
 P 2550 1100
-F 0 "#PWR?" H 2550 950 50  0001 C CNN
+F 0 "#PWR0112" H 2550 950 50  0001 C CNN
 F 1 "+24V" H 2565 1273 50  0000 C CNN
 F 2 "" H 2550 1100 50  0001 C CNN
@@
 	2550 1100 2300 1100
 $Comp
-L power:GND #PWR?
+L power:GND #PWR0113
 U 1 1 5FC11289
 P 2550 1300
-F 0 "#PWR?" H 2550 1050 50  0001 C CNN
+F 0 "#PWR0113" H 2550 1050 50  0001 C CNN
 F 1 "GND" H 2555 1127 50  0000 C CNN
 F 2 "" H 2550 1300 50  0001 C CNN
@@
 Induktiver Sensor LJ12 A3-4-Z/BX\n
 $Sheet
-S 4850 2100 1850 3900
-U 5FC14385
-F0 "Controller" 50
-F1 "Controller.sch" 50
+S 7600 3850 1200 900
+U 5FCAC453
+F0 "Stepper_y" 50
+F1 "Stepper_y.sch" 50
+F2 "CUR_CONTROL" I L 7600 3950 50
+F3 "STEP" I L 7600 4050 50
+F4 "DIR" I L 7600 4150 50
+F5 "DIAG" O L 7600 4250 50
+F6 "INDEX" O L 7600 4350 50
+F7 "SINGLE_WIRE" B L 7600 4450 50
+F8 "EN" I L 7600 4550 50
+F9 "OA1" O R 8800 4100 50
+F10 "OA2" O R 8800 4200 50
+F11 "OB1" O R 8800 4300 50
+F12 "OB2" O R 8800 4400 50
+$EndSheet
+$Sheet
+S 7600 2400 1200 900
+U 5FCAEEEC
+F0 "Stepper_z" 50
+F1 "Stepper_z.sch" 50
+F2 "CUR_CONTROL" I L 7600 2500 50
+F3 "STEP" I L 7600 2600 50
+F4 "DIR" I L 7600 2700 50
+F5 "DIAG" O L 7600 2800 50
+F6 "INDEX" O L 7600 2900 50
+F7 "SINGLE_WIRE" B L 7600 3000 50
+F8 "EN" I L 7600 3100 50
+F9 "OA1" O R 8800 2650 50
+F10 "OA2" O R 8800 2750 50
+F11 "OB1" O R 8800 2850 50
+F12 "OB2" O R 8800 2950 50
+$EndSheet
+$Sheet
+S 7600 1000 1200 900
+U 5FCB2242
+F0 "Stepper_rotation" 50
+F1 "Stepper_rotation.sch" 50
+F2 "CUR_CONTROL" I L 7600 1100 50
+F3 "STEP" I L 7600 1200 50
+F4 "DIR" I L 7600 1300 50
+F5 "DIAG" O L 7600 1400 50
+F6 "INDEX" O L 7600 1500 50
+F7 "SINGLE_WIRE" B L 7600 1600 50
+F8 "EN" I L 7600 1700 50
+F9 "OA1" O R 8800 1250 50
+F10 "OA2" O R 8800 1350 50
+F11 "OB1" O R 8800 1450 50
+F12 "OB2" O R 8800 1550 50
 $EndSheet
 $EndSCHEMATC

Commit message: STM32F401 für motoransteuerung gewählt. TODO: motoransteuerung und leistungsteil trennen, damit für schnelle fehlerbehebung modul getauscht werden kann
Parts:
- removed PS101: MEANWELL-MPM-90, pick_n_place:MEANWELL-MPM-90, symbol StepperBoard-rescue:MEANWELL-MPM-90-Pick_n_Place
- added C101, C104: 2.2u 50V, Capacitor_SMD:C_1210_3225Metric, symbol Device:C_Small
- added C102, C103: 18p 50V, Capacitor_SMD:C_0603_1608Metric, symbol Device:C_Small
- added C105, C106, C108, C111, C112, C115, C116: 10u 50V, Capacitor_SMD:C_1210_3225Metric, symbol Device:C_Small
- added C107, C109, C110, C113, C114: 100n 50V, Capacitor_SMD:C_0603_1608Metric, symbol Device:C_Small
- added FB101: 70R, Inductor_SMD:L_0603_1608Metric, symbol Device:Ferrite_Bead_Small
- added J106, J108: Conn_02x01, Connector_PinHeader_2.54mm:PinHeader_1x02_P2.54mm_Vertical, symbol Connector_Generic:Conn_02x01
- added J107: Conn_01x06_Male, Connector_PinHeader_2.54mm:PinHeader_1x06_P2.54mm_Vertical, symbol Connector:Conn_01x06_Male
- added J109: Micro_SD_Card_Det, ProjectFootprints:TF-115-BCP9, symbol StepperBoard:TF-115-BCP9
- added L101: 12u SRN4018, Inductor_SMD:L_Bourns-SRN4018, symbol Device:L_Small
- added R101: DNP, Resistor_SMD:R_0603_1608Metric, symbol Device:R_Small
- added R102, R103, R108, R109, R118: 10K, Resistor_SMD:R_0603_1608Metric, symbol Device:R_Small
- added R104, R105, R107: 51K, Resistor_SMD:R_0603_1608Metric, symbol Device:R_Small
- added R106, R112, R113, R114, R115, R116, R117: 22K1, Resistor_SMD:R_0603_1608Metric, symbol Device:R_Small
- added R110, R111: 100R, Resistor_SMD:R_0603_1608Metric, symbol Device:R_Small
- added U101: STM32F401VBTx, Package_QFP:LQFP-100_14x14mm_P0.5mm, symbol MCU_ST_STM32F4:STM32F401VBTx
- added U102: TPS560430, Package_TO_SOT_SMD:SOT-23-6, symbol StepperBoard:TPS560430
- added U103, U104: ST3485ECDR, Package_SO:SOIC-8_3.9x4.9mm_P1.27mm, symbol StepperBoard:THVD1500
- added Y101: 8MHz, Crystal:Crystal_SMD_3225-4Pin_3.2x2.5mm, symbol Device:Crystal_GND24
Connections:
- net +24V: now also J101.2 (Pin_2), C105.1, J106.1 (Pin_1)
- net GND: now also J101.1 (Pin_1), C101.2, C102.2, C103.2, C104.2, C105.2, C106.2, C107.2, C108.2, C109.2, C111.2, C112.2, C113.2, C114.2, C115.2, C116.2, J107.1 (Pin_1), J107.3 (Pin_3), J109.10 (SHIELD), J109.6 (VSS), R102.2, R105.1, R106.1, R108.2, R109.2, U101.10 (VSS), U101.20 (VSSA), U101.27 (VSS), U101.49 (VSS), U101.74 (VSS), U101.99 (VSS), U102.2 (GND), U103.5 (GND), U104.5 (GND), Y101.2, Y101.4
- new net: C102.1, U101.12 (PH0), Y101.1
- new net: C103.1, U101.13 (PH1), Y101.3
- new net: C101.1, U101.48 (VCAP1)
- new net: C104.1, U101.73 (VCAP2)
- new net: R101.1, R102.1, U101.94 (BOOT0)
- new net: C110.2, U102.1 (CB)
- new net: R106.2, R107.1, U102.3 (FB)
- new net: R104.2, R105.2, U102.4 (EN)
- new net: C106.1, C107.1, J106.2 (Pin_2), R104.1, U102.5 (Vin)
- new net: C110.1, L101.1, U102.6 (SW)
- new net: C111.1, C112.1, J108.1 (Pin_1), L101.2, R107.2
- new net +3V3: C113.1, C114.1, C115.1, C116.1, FB101.2, J108.2 (Pin_2), J109.4 (VDD), R101.2, R103.2, R112.2, R113.2, R114.2, R115.2, R116.2, R117.2, R118.1, U101.100 (VDD), U101.11 (VDD), U101.19 (VDD), U101.28 (VDD), U101.50 (VDD), U101.6 (VBAT), U101.75 (VDD), U103.8 (VCC), U104.8 (VCC)
- new net CAM_RS485+: R111.1, U104.7 (B)
- new net CAM_RS485-: R111.2, U104.6 (A)
- new net FEEDER_RS485+: R110.1, U103.7 (B)
- new net FEEDER_RS485-: R110.2, U103.6 (A)
- new net NRST: J107.5 (Pin_5), R103.1, U101.14 (NRST)
- new net PA10: U103.1 (R)
- new net PA13: J107.4 (Pin_4), U101.72 (PA13)
- new net PA14: J107.2 (Pin_2), U101.76 (PA14)
- new net PA15: J109.9 (DET_B), R118.2, U101.77 (PA15)
- new net PA8: R108.1, U103.2 (~RE), U103.3 (DE)
- new net PA9: U103.4 (D)
- new net PC10: J109.1 (DAT2), R117.1, U101.78 (PC10)
- new net PC11: J109.2 (DAT3/CD), R116.1, U101.79 (PC11)
- new net PC12: J109.5 (CLK), R114.1
- new net PC8: J109.7 (DAT0), R113.1, U101.65 (PC8)
- new net PC9: J109.8 (DAT1), R112.1, U101.66 (PC9)
- new net PD2: J109.3 (CMD), R115.1, U101.83 (PD2)
- new net PD4: R109.1, U101.85 (PD4), U104.2 (~RE), U104.3 (DE)
- new net PD5: U101.86 (PD5), U104.4 (D)
- new net PD6: U101.87 (PD6), U104.1 (R)
- new net VREF: C108.1, C109.1, FB101.1, U101.21 (VREF+), U101.22 (VDDA)
- no-connect marks 0 -> 1
Other:
- note added: "RS485 Receiver Transmitter"
- note added: "ST-LINK"
- moved on the sheet: J101, J102, J103, J104, J105
