File: Stepper_Modul/Stepper_xy.sch (KiCad schematic (older format))
At the start: 14 parts, among them SW301 SW_DIP_x03, U301 TMC2226

Commit message: motor controller von stepper-treibern getrennt, sodass es modular ist. Libraries werden nun übergreifend von allen projekten verwendet
Parts:
- removed C301, C305, C306, C307: 100n 50V, Capacitor_SMD:C_0603_1608Metric, symbol Device:C_Small
- removed C302, C303: 2.2u 50V, Capacitor_SMD:C_1210_3225Metric, symbol Device:C_Small
- removed C304: 22n 50V, Capacitor_SMD:C_0603_1608Metric, symbol Device:C_Small
- removed C308, C309: 100u 35V, Capacitor_THT:CP_Radial_D6.3mm_P2.50mm, symbol Device:CP_Small
- removed R301: 22k, Resistor_SMD:R_0603_1608Metric, symbol Device:R_Small
- removed R302, R303: 0.1R 0.5W, Resistor_SMD:R_1210_3225Metric, symbol Device:R_Small
- removed SW301: SW_DIP_x03, Package_DIP:DIP-6_W7.62mm, symbol Switch:SW_DIP_x03
- removed U301: TMC2226, Package_SO:TSSOP-28-1EP_4.4x9.7mm_P0.65mm, symbol StepperBoard-rescue:TMC2226-Pick_n_Place
- added C201, C205, C206, C207: 100n 50V, Capacitor_SMD:C_0603_1608Metric, symbol Device:C_Small
- added C202, C203: 2.2u 50V, Capacitor_SMD:C_1210_3225Metric, symbol Device:C_Small
- added C204: 22n 50V, Capacitor_SMD:C_0603_1608Metric, symbol Device:C_Small
- added C208, C209: 100u 35V, Capacitor_THT:CP_Radial_D6.3mm_P2.50mm, symbol Device:CP_Small
- added R201: 22k, Resistor_SMD:R_0603_1608Metric, symbol Device:R_Small
- added R202, R203: 0.22R 0.5W, Resistor_SMD:R_1210_3225Metric, symbol Device:R_Small
- added SW201: SW_DIP_x03, Package_DIP:DIP-6_W7.62mm, symbol Switch:SW_DIP_x03
- added U201: TMC2226, Package_SO:TSSOP-28-1EP_4.4x9.7mm_P0.65mm, symbol PorjectLibrary:TMC2226
Connections:
- net +24V: now also C205.2, C206.2, C207.2, C208.1, C209.1, U201.26 (VS), U201.3 (VS)
- net +3V3: now also C201.2, SW201.1, SW201.2, SW201.3, U201.19 (VCC_IO)
- net 5VOUT: now also C202.2, U201.11 (5VOUT)
- net GND: now also C201.1, C202.1, C203.1, C206.1, C207.1, C208.2, C209.2, R202.1, R203.1, U201.17 (CLK), U201.22 (GND), U201.24 (STDBY), U201.29 (GND), U201.6 (GND)
- net SINGLE_WIRE: now also U201.18 (PND_UART)
- new net: SW201.4, U201.10 (SPREAD)
- new net: SW201.6, U201.12 (MS1_AD0)
- new net: SW201.5, U201.14 (MS2_AD1)
- new net: R203.2, U201.2 (BRB)
- new net: C203.2, R201.1, U201.21 (VREF)
- new net: R202.2, U201.27 (BRA)
- new net: C204.2, U201.7 (CPO)
- new net: C204.1, U201.8 (CPI)
- new net: C205.1, U201.9 (VCP)
- new net CUR_CONTROL: R201.2
- new net DIAG: U201.15 (DIAG)
- new net DIR: U201.23 (DIR)
- new net EN: U201.5 (ENN)
- new net INDEX: U201.16 (INDEX)
- new net OA1: U201.28 (OA1)
- new net OA2: U201.25 (OA2)
- new net OB1: U201.1 (OB1)
- new net OB2: U201.4 (OB2)
- new net STEP: U201.20 (STEP)
Other:
- note added: "100mOhm C270892"
- note added: "960mA"
- note removed: "1920mA"
