File: Stepper_Modul/Stepper_x.sch (KiCad schematic (older format))
At the start: 14 parts, among them SW401 SW_DIP_x03, U401 TMC2226

Commit message: motor controller von stepper-treibern getrennt, sodass es modular ist. Libraries werden nun übergreifend von allen projekten verwendet
Parts:
- removed C401, C405, C406, C407: 100n 50V, Capacitor_SMD:C_0603_1608Metric, symbol Device:C_Small
- removed C402, C403: 2.2u 50V, Capacitor_SMD:C_1210_3225Metric, symbol Device:C_Small
- removed C404: 22n 50V, Capacitor_SMD:C_0603_1608Metric, symbol Device:C_Small
- removed C408, C409: 100u 35V, Capacitor_THT:CP_Radial_D6.3mm_P2.50mm, symbol Device:CP_Small
- removed R401: 22k, Resistor_SMD:R_0603_1608Metric, symbol Device:R_Small
- removed R402, R403: 0.1R 0.5W, Resistor_SMD:R_1210_3225Metric, symbol Device:R_Small
- removed SW401: SW_DIP_x03, Package_DIP:DIP-6_W7.62mm, symbol Switch:SW_DIP_x03
- removed U401: TMC2226, Package_SO:TSSOP-28-1EP_4.4x9.7mm_P0.65mm, symbol StepperBoard-rescue:TMC2226-Pick_n_Place
- added C201, C205, C206, C207: 100n 50V, Capacitor_SMD:C_0603_1608Metric, symbol Device:C_Small
- added C202, C203: 2.2u 50V, Capacitor_SMD:C_1210_3225Metric, symbol Device:C_Small
- added C204: 22n 50V, Capacitor_SMD:C_0603_1608Metric, symbol Device:C_Small
- added C208, C209: 100u 35V, Capacitor_THT:CP_Radial_D6.3mm_P2.50mm, symbol Device:CP_Small
- added R201: 22k, Resistor_SMD:R_0603_1608Metric, symbol Device:R_Small
- added R202, R203: 0.22R 0.5W, Resistor_SMD:R_1210_3225Metric, symbol Device:R_Small
- added SW201: SW_DIP_x03, Package_DIP:DIP-6_W7.62mm, symbol Switch:SW_DIP_x03
- added U201: TMC2226, Package_SO:TSSOP-28-1EP_4.4x9.7mm_P0.65mm, symbol PorjectLibrary:TMC2226
Connections:
- net +24V: now also C205.2, C206.2, C207.2, C208.1, C209.1, U201.26 (VS), U201.3 (VS)
- net +3V3: now also C201.2, SW201.1, SW201.2, SW201.3, U201.19 (VCC_IO)
- net 5VOUT: now also C202.2, U201.11 (5VOUT)
- net CUR_CONTROL_X: now also R201.2
- net DIAG_X: now also U201.15 (DIAG)
- net DIR_X: now also U201.23 (DIR)
- net EN_X: now also U201.5 (ENN)
- net GND: now also C201.1, C202.1, C203.1, C206.1, C207.1, C208.2, C209.2, R202.1, R203.1, U201.17 (CLK), U201.22 (GND), U201.24 (STDBY), U201.29 (GND), U201.6 (GND)
- net INDEX_X: now also U201.16 (INDEX)
- net OA1_X: now also U201.28 (OA1)
- net OA2_X: now also U201.25 (OA2)
- net OB1_X: now also U201.1 (OB1)
- net OB2_X: now also U201.4 (OB2)
- net SINGLE_WIRE: now also U201.18 (PND_UART)
- net STEP_X: now also U201.20 (STEP)
- new net: SW201.4, U201.10 (SPREAD)
- new net: SW201.6, U201.12 (MS1_AD0)
- new net: SW201.5, U201.14 (MS2_AD1)
- new net: R203.2, U201.2 (BRB)
- new net: C203.2, R201.1, U201.21 (VREF)
- new net: R202.2, U201.27 (BRA)
- new net: C204.2, U201.7 (CPO)
- new net: C204.1, U201.8 (CPI)
- new net: C205.1, U201.9 (VCP)
Other:
- note added: "100mOhm C270892"
- note added: "960mA"
- note removed: "1920mA"

Commit message: stepper board fertig gestellt
Parts:
- R201: value 22k -> 22K1; LCSC C31850 -> C137768
Changed lines of the file:
@@
 AR Path="/5FCAC453/5FBDD375" Ref="R504"  Part="1"
 F 0 "R504" V 5114 950 50  0000 C CNN
-F 1 "22k" V 5205 950 50  0000 C CNN
+F 1 "22K1" V 5205 950 50  0000 C CNN
 F 2 "Resistor_SMD:R_0603_1608Metric" H 5400 950 50  0001 C CNN
 F 3 "~" H 5400 950 50  0001 C CNN
-F 4 "C31850" V 5296 950 50  0000 C CNN "LCSC"
+F 4 "C137768" V 5296 950 50  0000 C CNN "LCSC"
 	1    5400 950
 	0    1    1    0

Commit message: BOM für LCSC überarbeitet. Tool für BOM export modifiziert
Parts:
- C208, C209: LCSC C156874 -> C45075
Changed lines of the file:
@@
 F 2 "Capacitor_THT:CP_Radial_D6.3mm_P2.50mm" H 8900 2200 50  0001 C CNN
 F 3 "https://datasheet.lcsc.com/szlcsc/Guangdong-TOPAZ-Elec-Tech-ECSS0608101M035P00_C156874.pdf" H 8900 2200 50  0001 C CNN
-F 4 "C156874" H 8988 2109 50  0000 L CNN "LCSC"
+F 4 "C45075" H 8988 2109 50  0000 L CNN "LCSC"
 	1    8900 2200
 	1    0    0    -1
@@
 F 2 "Capacitor_THT:CP_Radial_D6.3mm_P2.50mm" H 9450 2200 50  0001 C CNN
 F 3 "https://datasheet.lcsc.com/szlcsc/Guangdong-TOPAZ-Elec-Tech-ECSS0608101M035P00_C156874.pdf" H 9450 2200 50  0001 C CNN
-F 4 "C156874" H 9538 2109 50  0000 L CNN "LCSC"
+F 4 "C45075" H 9538 2109 50  0000 L CNN "LCSC"
 	1    9450 2200
 	1    0    0    -1
