File: Stepper_Modul/Stepper_z.sch (KiCad schematic (older format))
At the start: 14 parts, among them SW401 SW_DIP_x03, U401 TMC2226

Commit message: stepper board fertig gestellt
Parts:
- R401: value 22k -> 22K1; LCSC C31850 -> C137768
Changed lines of the file:
@@
 AR Path="/5FCB2242/5FCB624B" Ref="R?"  Part="1"
 F 0 "R401" V 5114 950 50  0000 C CNN
-F 1 "22k" V 5205 950 50  0000 C CNN
+F 1 "22K1" V 5205 950 50  0000 C CNN
 F 2 "Resistor_SMD:R_0603_1608Metric" H 5400 950 50  0001 C CNN
 F 3 "~" H 5400 950 50  0001 C CNN
-F 4 "C31850" V 5296 950 50  0000 C CNN "LCSC"
+F 4 "C137768" V 5296 950 50  0000 C CNN "LCSC"
 	1    5400 950
 	0    1    1    0

Commit message: BOM für LCSC überarbeitet. Tool für BOM export modifiziert
Parts:
- C408, C409: LCSC C156874 -> C45075
Changed lines of the file:
@@
 F 2 "Capacitor_THT:CP_Radial_D6.3mm_P2.50mm" H 8900 2200 50  0001 C CNN
 F 3 "https://datasheet.lcsc.com/szlcsc/Guangdong-TOPAZ-Elec-Tech-ECSS0608101M035P00_C156874.pdf" H 8900 2200 50  0001 C CNN
-F 4 "C156874" H 8988 2109 50  0000 L CNN "LCSC"
+F 4 "C45075" H 8988 2109 50  0000 L CNN "LCSC"
 	1    8900 2200
 	1    0    0    -1
@@
 F 2 "Capacitor_THT:CP_Radial_D6.3mm_P2.50mm" H 9450 2200 50  0001 C CNN
 F 3 "https://datasheet.lcsc.com/szlcsc/Guangdong-TOPAZ-Elec-Tech-ECSS0608101M035P00_C156874.pdf" H 9450 2200 50  0001 C CNN
-F 4 "C156874" H 9538 2109 50  0000 L CNN "LCSC"
+F 4 "C45075" H 9538 2109 50  0000 L CNN "LCSC"
 	1    9450 2200
 	1    0    0    -1

Commit message: Änderungen für bestellung V01 -  Bestellung abgeschickt
Parts:
- R402, R403: value 0.1R 0.5W -> 0.5R 0.5W; LCSC C270892 -> C305329
Changed lines of the file:
@@
 AR Path="/5FCB2242/5FCB6236" Ref="R?"  Part="1"
 F 0 "R402" V 7714 3200 50  0000 C CNN
-F 1 "0.1R 0.5W" V 7805 3200 50  0000 C CNN
+F 1 "0.5R 0.5W" V 7805 3200 50  0000 C CNN
 F 2 "Resistor_SMD:R_1210_3225Metric" H 8000 3200 50  0001 C CNN
 F 3 "~" H 8000 3200 50  0001 C CNN
-F 4 "C270892" V 7896 3200 50  0000 C CNN "LCSC"
+F 4 "C305329" V 7896 3200 50  0000 C CNN "LCSC"
 	1    8000 3200
 	0    1    1    0
@@
 AR Path="/5FCB2242/5FCB6238" Ref="R?"  Part="1"
 F 0 "R403" V 7714 3850 50  0000 C CNN
-F 1 "0.1R 0.5W" V 7805 3850 50  0000 C CNN
+F 1 "0.5R 0.5W" V 7805 3850 50  0000 C CNN
 F 2 "Resistor_SMD:R_1210_3225Metric" H 8000 3850 50  0001 C CNN
 F 3 "~" H 8000 3850 50  0001 C CNN
-F 4 "C270892" V 7896 3850 50  0000 C CNN "LCSC"
+F 4 "C305329" V 7896 3850 50  0000 C CNN "LCSC"
 	1    8000 3850
 	0    1    1    0
