File: Feeder_Modul/RepoPNP/KiCad/4_Wall/Wall_F_V4/Wall-F_V3.sch (KiCad schematic (older format))
At the start: 55 parts, among them J1 Conn_01x01, J10 H-Bridge, J12 SW_ENC_LED, J15 Daisy, J16 Conn_01x01, J17 Conn_01x01, J2 Daisy, J3 PWR, J5 Conn_01x01, J7 SWD Interface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

Commit message: Schaltplan für Feeder fast fertig, Wichtige Komponenten auf der PCB geplaced. DXF Outline und Annotations für Bauteile konnten erfolgreich importiert werden
Parts:
- C1, C2: symbol CP -> Wall-F_V3-rescue:CP
- C10, C11, C12, C13, C14, C15, C16, C17, C3, C4, C5, C6, C7, C8, C9: symbol C -> Wall-F_V3-rescue:C
- D1: symbol LED -> Wall-F_V3-rescue:LED
- D2: symbol D_Schottky_x2_ACom_AKK -> Wall-F_V3-rescue:D_Schottky_x2_ACom_AKK
- J1, J16, J17, J5: symbol Conn_01x01 -> Wall-F_V3-rescue:Conn_01x01
- J10: symbol Conn_01x05 -> Wall-F_V3-rescue:Conn_01x05
- J12: symbol Conn_01x06 -> Wall-F_V3-rescue:Conn_01x06
- J15, J2: symbol Conn_02x03_Odd_Even -> Wall-F_V3-rescue:Conn_02x03_Odd_Even
- J3, J8, J9: symbol Conn_01x02 -> Wall-F_V3-rescue:Conn_01x02
- J7: symbol Conn_02x05_Odd_Even -> Wall-F_V3-rescue:Conn_02x05_Odd_Even
- L1: symbol Ferrite_Bead_Small -> Wall-F_V3-rescue:Ferrite_Bead_Small
- Q1: symbol BC847 -> Wall-F_V3-rescue:BC847
- R1, R10, R11, R12, R14, R2, R5, R6, R7, R8, R9: symbol R -> Wall-F_V3-rescue:R
- SW1, SW2, SW3, SW4: symbol SW_Push -> Wall-F_V3-rescue:SW_Push
- U1, U3: symbol EE-SX1350_PCB -> Wall-F_V3-rescue:EE-SX1350_PCB
- U2: symbol DRV8835 -> Wall-F_V3-rescue:DRV8835
- U4: symbol MK20DX128VFT -> Wall-F_V3-rescue:MK20DX128VFT
- U5: symbol TC1262-33 -> Wall-F_V3-rescue:TC1262-33
- Y1: symbol Crystal_GND24 -> Wall-F_V3-rescue:Crystal_GND24
- Y2: symbol Crystal -> Wall-F_V3-rescue:Crystal
