File: Controller_Modul/Controller_Modul.sch (KiCad schematic (older format))
At the start: 46 parts

Commit message: Conroller Modul Schaltplan fertig
Parts:
- removed C? (x2): 100n 50V, Capacitor_SMD:C_0603_1608Metric, symbol Device:C_Small
- removed R? (x2): 100R, Resistor_SMD:R_0603_1608Metric, symbol Device:R_Small
- removed R? (x2): 10K, Resistor_SMD:R_0603_1608Metric, symbol Device:R_Small
- removed U?: STM32F401VBTx, Package_QFP:LQFP-100_14x14mm_P0.5mm, symbol MCU_ST_STM32F4:STM32F401VBTx
- removed U? (x2): ST3485ECDR, Package_SO:SOIC-8_3.9x4.9mm_P1.27mm, symbol PorjectLibrary:THVD1500
- added C113, C114, C115, C116, C117, C118: 100n, Capacitor_SMD:C_0603_1608Metric, symbol Device:C_Small
- added C119, C120: 10u, Capacitor_SMD:C_1210_3225Metric, symbol Device:C_Small
- added D101: SS22F-SS2200F, Diode_SMD:D_SMA, symbol Device:D_Schottky_Small
- added J105: Conn_01x04_Male, Connector_PinHeader_2.54mm:PinHeader_1x04_P2.54mm_Vertical, symbol Connector:Conn_01x04_Male
- added J106: Conn_01x08_Male, ProjectFootprints:ST7789_Waveshare, symbol Connector:Conn_01x08_Male
- added J108: Screw_Terminal_01x04, TerminalBlock_RND:TerminalBlock_RND_205-00047_1x04_P5.00mm_Horizontal, symbol Connector:Screw_Terminal_01x04
- added J109, J111: Conn_02x20_Odd_Even, Connector_PinHeader_2.54mm:PinHeader_2x20_P2.54mm_Vertical, symbol Connector_Generic:Conn_02x20_Odd_Even
- added J110: USB_B_Mini, Connector_USB:USB_B_OST_USB-B1HSxx_Horizontal, symbol PorjectLibrary:USB_B
- added L102, L103: DNP, ProjectFootprints:L_CommonModeChoke_Coilcraft_1812CAN, symbol Device:L_Core_Ferrite_Coupled
- added R101, R103, R104, R105, R106, R108, R109, R110, R111, R112, R113, R114, R115, R116, R117, R118, R119, R123, R124, R125, R126, R128, R129, R130, R132, R133, R136, R137, R138, R139, R155, R156, R157, R158, R159, R160, R161, R162, R163, R164, R165, R166, R167, R168, R169, R170, R171, R172, R173, R174, R175, R176, R177, R178, R179: 1K, Resistor_SMD:R_0603_1608Metric, symbol Device:R_Small
- added R134, R135, R140, R141: 10K, Resistor_SMD:R_0603_1608Metric, symbol Device:R_Small
- added R147, R148, R149, R150: 0R, Resistor_SMD:R_0603_1608Metric, symbol Device:R_Small
- added R153, R154: 120R, Resistor_SMD:R_0603_1608Metric, symbol Device:R_Small
- added SW101: Rotary_Encoder_Switch, Rotary_Encoder:RotaryEncoder_Alps_EC11E-Switch_Vertical_H20mm_CircularMountingHoles, symbol Device:Rotary_Encoder_Switch
- added U101: STM32F446VCTx, Package_QFP:LQFP-100_14x14mm_P0.5mm, symbol MCU_ST_STM32F4:STM32F446VCTx
- added U103, U104: SN65HVD230DR, Package_SO:SOIC-8_3.9x4.9mm_P1.27mm, symbol Interface_CAN_LIN:TJA1051T-3
- gave numbers to parts that had none: 37
Connections:
- net labels added: ADC_RES1, ADC_RES2, ADC_RES3, ADC_RES4, CAN1_H, CAN1_L, CAN1_RX, CAN1_TX, CAN2_H, CAN2_L, CAN2_RX, CAN2_TX, CUR_ROT, CUR_X, CUR_Y, CUR_Z, DIAG_ROT, DIAG_X, DIAG_Y, DIAG_Z, DIR_ROT, DIR_X, DIR_Y, DIR_Z, DISP_BL, DISP_CLK, DISP_CS, DISP_DC, DISP_DIN, DISP_RST, ENC_BTN, ENDSTEP_Z1, ENDSTOP_ROT1, ENDSTOP_ROT2, ENDSTOP_X1, ENDSTOP_X2, ENDSTOP_Y1, ENDSTOP_Y2, ENDSTOP_Z2, EN_ROT, EN_X, EN_Y, EN_Z, I2C1_SCL, I2C1_SDA, INDEX_ROT, INDEX_X, INDEX_Y, INDEX_Z, INPUT_RES1, INPUT_RES2, OUTPUT_RES1, OUTPUT_RES2, OUTPUT_RES3, OUTPUT_RES4, OUTPUT_RES5, OUTPUT_RES6, OUTPUT_RES7, PA0, PA1, PA11, PA12, PA2, PA3, PA4, PA5, PA6, PB0, PB1, PB10, PB12, PB13, PB14, PB15, PB2, PB3, PB4, PB5, PB6, PB7, PB8, PB9, PC0, PC1, PC13, PC14, PC15, PC2, PC3, PC4, PC5, PC6, PC7, PD0, PD1, PD10, PD11, PD12, PD13, PD14, PD15, PD3, PD7, PD8, PD9, PE0, PE1, PE10, PE11, PE12, PE13, PE2, PE3, PE4, PE5, PE6, PE7, PE9, SINGLE_WIRE, SPI1_SCK, SPI_MOSI, STEP_ROT, STEP_X, STEP_Y, STEP_Z, TIM1_CH1_Z, TIM2_CH1_X, TIM3_CH1_ROT, TIM4_CH1, TIM4_CH2, TIM4_CH3, TIM4_CH4, TIM5_CH1_Y, TIM8_ENC_CH1, TIM8_ENC_CH2, USB_FS_DM, USB_FS_DP, VACUUM_MOTOR, VENTIL1, VENTIL2
- net labels removed: CAM_RS485+, CAM_RS485-, FEEDER_RS485+, FEEDER_RS485-, RX2, Rx1, RxTx1_DIR, RxTx2_DIR, TX2, Tx1
- wire segments 176 -> 404
- no-connect marks 1 -> 6
Other:
- note added: "Connector to plug Nintendo Nunchuck"
- note added: "Replacement\nTJA1051T-3"
- note added: "Waveshare 2inch ST7789 Display"
- note removed: "Induktiver Sensor LJ12 A3-4-Z/BX\n"
- note removed: "RS485 Receiver Transmitter"
- moved on the sheet: C101, C102, C103, C104, C108, C109, C121, C122, FB101, J101, J103, J107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

Commit message: Controller Board geplaced
Parts:
- removed J101: Screw_Terminal_01x02, TerminalBlock_RND:TerminalBlock_RND_205-00045_1x02_P5.00mm_Horizontal, symbol Connector:Screw_Terminal_01x02
- removed J108: Screw_Terminal_01x04, TerminalBlock_RND:TerminalBlock_RND_205-00047_1x04_P5.00mm_Horizontal, symbol Connector:Screw_Terminal_01x04
- added C123, C124, C125, C126, C127, C128, C129: 100n 50V, Capacitor_SMD:C_0603_1608Metric, symbol Device:C_Small
- added H101, H102, H103, H104: MountingHole_Pad, MountingHole:MountingHole_3.2mm_M3_Pad_Via, symbol Mechanical:MountingHole_Pad
- added J101: Screw_Terminal_01x06, TerminalBlock_RND:TerminalBlock_RND_205-00049_1x06_P5.00mm_Horizontal, symbol Connector:Screw_Terminal_01x06
- added J108: Conn_02x07_Odd_Even, Connector_PinHeader_2.54mm:PinHeader_2x07_P2.54mm_Vertical, symbol Connector_Generic:Conn_02x07_Odd_Even
Connections:
- net +3V3: now also C123.2, C124.1, C125.2, C126.1, C127.2, C128.1, C129.2, J108.1 (Pin_1)
- net CAN1_H: now also L102.2, J101.3 (Pin_3); no longer L102.1
- net CAN1_L: now also L102.4, J101.4 (Pin_4); no longer L102.3
- net CAN2_H: now also L103.2, J101.5 (Pin_5); no longer L103.1
- net CAN2_L: now also L103.4, J101.6 (Pin_6); no longer L103.3
- net DISP_BL: now also J108.9 (Pin_9)
- net DISP_CLK: now also J108.4 (Pin_4)
- net DISP_CS: now also J108.5 (Pin_5)
- net DISP_DC: now also J108.6 (Pin_6)
- net DISP_DIN: now also J108.3 (Pin_3)
- net DISP_RST: now also J108.7 (Pin_7), J108.8 (Pin_8)
- net ENC_BTN: now also J108.14 (Pin_14)
- net GND: now also C123.1, C124.2, C125.1, C126.2, C127.1, C128.2, C129.1, H101.1, H102.1, H103.1, H104.1, J101.2 (Pin_2), J108.10 (Pin_10), J108.12 (Pin_12), J108.2 (Pin_2)
- net PC6: now also J108.13 (Pin_13)
- net PC7: now also J108.11 (Pin_11)
- net at D101.2 (A): now also J101.1 (Pin_1)
- net at R148.1, U103.6 (CANL): now also L102.3; no longer L102.4
- net at R147.2, U103.7 (CANH): now also L102.1; no longer L102.2
- net at R150.1, U104.6 (CANL): now also L103.3; no longer L103.4
- net at R149.2, U104.7 (CANH): now also L103.1; no longer L103.2
Other:
- moved on the sheet: D101

Commit message: Controller Modul und CV Modul Can schaltung berichtigt. CV Modul abgerundete Ecken r=5mm. TODO: IO Modul, Feeder-Steckplätze, Display Modul
Parts:
- removed C115, C116: 100n, Capacitor_SMD:C_0603_1608Metric, symbol Device:C_Small
- removed U103, U104: SN65HVD230DR, Package_SO:SOIC-8_3.9x4.9mm_P1.27mm, symbol Interface_CAN_LIN:TJA1051T-3
- added J112, J113: Conn_02x01, Connector_PinHeader_2.54mm:PinHeader_1x02_P2.54mm_Vertical, symbol Connector_Generic:Conn_02x01
- added R180, R181: DNP, Resistor_SMD:R_0603_1608Metric, symbol Device:R_Small
- added U103, U104: SN65HVD230, Package_SO:SOIC-8_3.9x4.9mm_P1.27mm, symbol Interface_CAN_LIN:SN65HVD230
Connections:
- net +3V3: now also R180.1, R181.1, U103.3 (VCC), U104.3 (VCC); no longer R140.1, R141.1
- net CAN1_L: now also J112.2 (Pin_2); no longer R153.2
- net CAN1_RX: now also U103.4 (R)
- net CAN1_TX: now also U103.1 (D)
- net CAN2_L: now also J113.2 (Pin_2); no longer R154.2
- net CAN2_RX: now also U104.4 (R)
- net CAN2_TX: now also U104.1 (D)
- net GND: now also R140.2, R141.2, U103.2 (GND), U104.2 (GND)
- net at L102.3, R148.1: now also U103.6 (CANL)
- net at L102.1, R147.2: now also U103.7 (CANH)
- net at L103.3, R150.1: now also U104.6 (CANL)
- net at L103.1, R149.2: now also U104.7 (CANH)
- new net: J112.1 (Pin_1), R153.2
- new net: R140.1, R180.2, U103.8 (Rs)
- new net: R141.1, R181.2, U104.8 (Rs)
- new net: J113.1 (Pin_1), R154.2
- no-connect marks 6 -> 8
Other:
- note added: "Built in ESD Protection 16kV"
- note added: "High Speed Mode"
- note removed: "Replacement\nTJA1051T-3"
- moved on the sheet: R140, R141, R153, R154
