File: Controller_Modul/Controller_Modul.sch (KiCad schematic (older format))
At the start: 147 parts, among them J101 Screw_Terminal_01x06, J102 Conn_02x01, J103 Conn_01x06_Male, J104 Conn_02x01, J105 Conn_01x04_Male, J106 Conn_01x08_Male, J107 Micro_SD_Card_Det, J108 IPC 16P, J109 Conn_02x20_Odd_Even, J110 USB_B_Mini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

Commit message: Änderungen für bestellung V01 -  Bestellung abgeschickt
Parts:
- FID101, FID102, FID103: LCSC (none) -> 0
Connections:
- net USB_FS_D+: now also U105.6 (IO4); no longer U105.4 (IO3)
- net USB_FS_D-: now also U105.4 (IO3); no longer U105.6 (IO4)
Other:
- note removed: "TODO: Length Matching SDIO, SPI beachten\nConnector für Display mit CPU-Board abstimmen\nESD Schutz USB-Buchse\nStatus LED"
Changed lines of the file:
@@
 Wire Wire Line
 	9400 9650 9400 9550
-Text Notes 5350 6750 0    129  ~ 0
-TODO: Length Matching SDIO, SPI beachten\nConnector für Display mit CPU-Board abstimmen\nESD Schutz USB-Buchse\nStatus LED
 $Comp
 L Power_Protection:SRV05-4 U105
@@
 $EndComp
 Text Label 7250 3550 0    50   ~ 0
-USB_FS_D+
-Text Label 7250 3750 0    50   ~ 0
 USB_FS_D-
 $Comp
@@
 F 2 "Fiducial:Fiducial_1mm_Mask2mm" H 6500 10500 50  0001 C CNN
 F 3 "~" H 6500 10500 50  0001 C CNN
+F 4 "0" H 6500 10500 50  0001 C CNN "LCSC"
 	1    6500 10500
 	1    0    0    -1
@@
 F 2 "Fiducial:Fiducial_1mm_Mask2mm" H 7000 10500 50  0001 C CNN
 F 3 "~" H 7000 10500 50  0001 C CNN
+F 4 "0" H 7000 10500 50  0001 C CNN "LCSC"
 	1    7000 10500
 	1    0    0    -1
@@
 F 2 "Fiducial:Fiducial_1mm_Mask2mm" H 7500 10500 50  0001 C CNN
 F 3 "~" H 7500 10500 50  0001 C CNN
+F 4 "0" H 7500 10500 50  0001 C CNN "LCSC"
 	1    7500 10500
 	1    0    0    -1
@@
 Wire Wire Line
 	13850 1850 14550 1850
+Text Label 7250 3750 0    50   ~ 0
+USB_FS_D+
 $EndSCHEMATC
