File: FeederRail_Modul/FeederRail_Modul.sch (KiCad schematic (older format))
At the start: 50 parts, among them J101 Conn_02x07_Odd_Even, J102 Conn_02x07_Odd_Even, J103 Conn_02x07_Odd_Even, J104 Conn_02x07_Odd_Even, J105 Conn_02x07_Odd_Even

Commit message: Feeder Rail mit Step files geprüft. Connector am Feeder verschoeben. Halter für Lager muss angepasst werden.
Parts:
- J101, J102, J103, J104, J105: footprint Connector_PinHeader_2.54mm:PinHeader_2x08_P2.54mm_Vertical -> ProjectFootprints:PinHeader_2x08_P2.54mm_Vertical
Changed lines of the file:
@@
 F 0 "J102" H 2100 1867 50  0000 C CNN
 F 1 "Conn_02x07_Odd_Even" H 2100 1776 50  0000 C CNN
-F 2 "Connector_PinHeader_2.54mm:PinHeader_2x08_P2.54mm_Vertical" H 2050 1350 50  0001 C CNN
+F 2 "ProjectFootprints:PinHeader_2x08_P2.54mm_Vertical" H 2050 1350 50  0001 C CNN
 F 3 "~" H 2050 1350 50  0001 C CNN
 F 4 "C30734" H 2050 1350 50  0001 C CNN "LCSC"
@@
 F 0 "J101" H 2050 3367 50  0000 C CNN
 F 1 "Conn_02x07_Odd_Even" H 2050 3276 50  0000 C CNN
-F 2 "Connector_PinHeader_2.54mm:PinHeader_2x08_P2.54mm_Vertical" H 2000 2850 50  0001 C CNN
+F 2 "ProjectFootprints:PinHeader_2x08_P2.54mm_Vertical" H 2000 2850 50  0001 C CNN
 F 3 "~" H 2000 2850 50  0001 C CNN
 F 4 "C30734" H 2000 2850 50  0001 C CNN "LCSC"
@@
 F 0 "J104" H 5600 3367 50  0000 C CNN
 F 1 "Conn_02x07_Odd_Even" H 5600 3276 50  0000 C CNN
-F 2 "Connector_PinHeader_2.54mm:PinHeader_2x08_P2.54mm_Vertical" H 5550 2850 50  0001 C CNN
+F 2 "ProjectFootprints:PinHeader_2x08_P2.54mm_Vertical" H 5550 2850 50  0001 C CNN
 F 3 "~" H 5550 2850 50  0001 C CNN
 F 4 "C30734" H 5550 2850 50  0001 C CNN "LCSC"
@@
 F 0 "J103" H 2100 4817 50  0000 C CNN
 F 1 "Conn_02x07_Odd_Even" H 2100 4726 50  0000 C CNN
-F 2 "Connector_PinHeader_2.54mm:PinHeader_2x08_P2.54mm_Vertical" H 2050 4300 50  0001 C CNN
+F 2 "ProjectFootprints:PinHeader_2x08_P2.54mm_Vertical" H 2050 4300 50  0001 C CNN
 F 3 "~" H 2050 4300 50  0001 C CNN
 F 4 "C30734" H 2050 4300 50  0001 C CNN "LCSC"
@@
 F 0 "J105" H 5650 1817 50  0000 C CNN
 F 1 "Conn_02x07_Odd_Even" H 5650 1726 50  0000 C CNN
-F 2 "Connector_PinHeader_2.54mm:PinHeader_2x08_P2.54mm_Vertical" H 5600 1300 50  0001 C CNN
+F 2 "ProjectFootprints:PinHeader_2x08_P2.54mm_Vertical" H 5600 1300 50  0001 C CNN
 F 3 "~" H 5600 1300 50  0001 C CNN
 F 4 "C30734" H 5600 1300 50  0001 C CNN "LCSC"
